File: Proto_Nano.sch (KiCad schematic (older format))
At the start: 32 parts, among them J1 USB_OTG, J2 ICSP_Header, SW1 RESET, U1 LM1117-5.0, U2 CH340G, U3 ATMEGA328P-AU, Y1 12MHz, Y2 16MHz

Commit message: fix a Thing on the schematic replace the symbol for the ICSP header with a more logical one, and move it to a different place in the schematic
Parts:
- removed J2: ICSP_Header, Pin_Headers:Pin_Header_Straight_2x03_Pitch2.54mm, symbol ICSP_Header-RESCUE-Proto_Nano
- removed U1: LM1117-5.0, TO_SOT_Packages_SMD:SOT-223, symbol LM1117-SMD
- added J?: ICSP_Header_Slave, Pin_Headers:Pin_Header_Straight_2x03_Pitch2.54mm, symbol ICSP_Header_Slave
- added U?: LM1117, symbol LM1117
Connections:
- wire segments 63 -> 85
Other:
- note added: "In-Circuit\nSerial\nProgramming\nHeader"
- note removed: "In-Circuit Serial\nProgramming Header"
- moved on the sheet: C10, D2, D3, D4, D5, R1, R2, R3, R4, R5, R6, R7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
